File: PCB/keyboard-1/tenet-kb-1.kicad_sch (KiCad schematic)
At the start: 14 parts, among them SW1 SW_Push, U1 ATmega32U4-A, Y1 16MHz

Commit message: keyswitch schematics
Parts:
- added D1, D10, D11, D12, D13, D14, D15, D16, D17, D18, D19, D2, D20, D21, D22, D23, D24, D25, D26, D27, D28, D29, D3, D30, D31, D32, D33, D34, D35, D36, D37, D38, D39, D4, D40, D41, D42, D43, D44, D45, D46, D47, D48, D49, D5, D50, D6, D7, D8, D9: D_Small, symbol Device:D_Small
- added MX1: K_A1, symbol MX_Alps_Hybrid:MX-NoLED
- added MX10: K_C2, symbol MX_Alps_Hybrid:MX-NoLED
- added MX11: K_C3, symbol MX_Alps_Hybrid:MX-NoLED
- added MX12: K_C4, symbol MX_Alps_Hybrid:MX-NoLED
- added MX13: K_D1, symbol MX_Alps_Hybrid:MX-NoLED
- added MX14: K_D2, symbol MX_Alps_Hybrid:MX-NoLED
- added MX15: K_D3, symbol MX_Alps_Hybrid:MX-NoLED
- added MX16: K_D4, symbol MX_Alps_Hybrid:MX-NoLED
- added MX17: K_E1, symbol MX_Alps_Hybrid:MX-NoLED
- added MX18: K_E2, symbol MX_Alps_Hybrid:MX-NoLED
- added MX19: K_E3, symbol MX_Alps_Hybrid:MX-NoLED
- added MX2: K_A2, symbol MX_Alps_Hybrid:MX-NoLED
- added MX20: K_E4, symbol MX_Alps_Hybrid:MX-NoLED
- added MX21: K_F1, symbol MX_Alps_Hybrid:MX-NoLED
- added MX22: K_F2, symbol MX_Alps_Hybrid:MX-NoLED
- added MX23: K_F3, symbol MX_Alps_Hybrid:MX-NoLED
- added MX24: K_F4, symbol MX_Alps_Hybrid:MX-NoLED
- added MX25: K_G4, symbol MX_Alps_Hybrid:MX-NoLED
- added MX26: K_I1, symbol MX_Alps_Hybrid:MX-NoLED
- added MX27: K_I2, symbol MX_Alps_Hybrid:MX-NoLED
- added MX28: K_I3, symbol MX_Alps_Hybrid:MX-NoLED
- added MX29: K_I4, symbol MX_Alps_Hybrid:MX-NoLED
- added MX3: K_A3, symbol MX_Alps_Hybrid:MX-NoLED
- added MX30: K_J1, symbol MX_Alps_Hybrid:MX-NoLED
- added MX31: K_J2, symbol MX_Alps_Hybrid:MX-NoLED
- added MX32: K_J3, symbol MX_Alps_Hybrid:MX-NoLED
- added MX33: K_J4, symbol MX_Alps_Hybrid:MX-NoLED
- added MX34: K_K1, symbol MX_Alps_Hybrid:MX-NoLED
- added MX35: K_K2, symbol MX_Alps_Hybrid:MX-NoLED
- added MX36: K_K3, symbol MX_Alps_Hybrid:MX-NoLED
- added MX37: K_K4, symbol MX_Alps_Hybrid:MX-NoLED
- added MX38: K_L1, symbol MX_Alps_Hybrid:MX-NoLED
- added MX39: K_L2, symbol MX_Alps_Hybrid:MX-NoLED
- added MX4: K_A4, symbol MX_Alps_Hybrid:MX-NoLED
- added MX40: K_L3, symbol MX_Alps_Hybrid:MX-NoLED
- added MX41: K_L4, symbol MX_Alps_Hybrid:MX-NoLED
- added MX42: K_M1, symbol MX_Alps_Hybrid:MX-NoLED
- added MX43: K_M2, symbol MX_Alps_Hybrid:MX-NoLED
- added MX44: K_M3, symbol MX_Alps_Hybrid:MX-NoLED
- added MX45: K_M4, symbol MX_Alps_Hybrid:MX-NoLED
- added MX46: K_N1, symbol MX_Alps_Hybrid:MX-NoLED
- added MX47: K_N2, symbol MX_Alps_Hybrid:MX-NoLED
- added MX48: K_N3, symbol MX_Alps_Hybrid:MX-NoLED
- added MX49: K_N4, symbol MX_Alps_Hybrid:MX-NoLED
- added MX5: K_B1, symbol MX_Alps_Hybrid:MX-NoLED
- added MX50: K_H4, symbol MX_Alps_Hybrid:MX-NoLED
- added MX6: K_B2, symbol MX_Alps_Hybrid:MX-NoLED
- added MX7: K_B3, symbol MX_Alps_Hybrid:MX-NoLED
- added MX8: K_B4, symbol MX_Alps_Hybrid:MX-NoLED
- added MX9: K_C1, symbol MX_Alps_Hybrid:MX-NoLED
Connections:
- new net: D36.2 (A), MX36.2 (ROW)
- new net: D35.2 (A), MX35.2 (ROW)
- new net: D5.2 (A), MX5.2 (ROW)
- new net: D41.2 (A), MX41.2 (ROW)
- new net: D6.2 (A), MX6.2 (ROW)
- new net: D29.2 (A), MX29.2 (ROW)
- new net: D9.2 (A), MX9.2 (ROW)
- new net: D20.2 (A), MX20.2 (ROW)
- new net: D46.2 (A), MX46.2 (ROW)
- new net: D24.2 (A), MX24.2 (ROW)
- new net: D14.2 (A), MX14.2 (ROW)
- new net: D21.2 (A), MX21.2 (ROW)
- new net: D31.2 (A), MX31.2 (ROW)
- new net: D16.2 (A), MX16.2 (ROW)
- new net: D27.2 (A), MX27.2 (ROW)
- new net: D48.2 (A), MX48.2 (ROW)
- new net: D43.2 (A), MX43.2 (ROW)
- new net: D22.2 (A), MX22.2 (ROW)
- new net: D30.2 (A), MX30.2 (ROW)
- new net: D28.2 (A), MX28.2 (ROW)
- new net: D17.2 (A), MX17.2 (ROW)
- new net: D12.2 (A), MX12.2 (ROW)
- new net: D38.2 (A), MX38.2 (ROW)
- new net: D13.2 (A), MX13.2 (ROW)
- new net: D33.2 (A), MX33.2 (ROW)
- new net: D18.2 (A), MX18.2 (ROW)
- new net: D45.2 (A), MX45.2 (ROW)
- new net: D40.2 (A), MX40.2 (ROW)
- new net: D32.2 (A), MX32.2 (ROW)
- new net: D47.2 (A), MX47.2 (ROW)
- new net: D7.2 (A), MX7.2 (ROW)
- new net: D26.2 (A), MX26.2 (ROW)
- new net: D25.2 (A), MX25.2 (ROW)
- new net: D8.2 (A), MX8.2 (ROW)
- new net: D11.2 (A), MX11.2 (ROW)
- new net: D39.2 (A), MX39.2 (ROW)
- new net: D49.2 (A), MX49.2 (ROW)
- new net: D34.2 (A), MX34.2 (ROW)
- new net: D2.2 (A), MX2.2 (ROW)
- new net: D4.2 (A), MX4.2 (ROW)
- new net: D15.2 (A), MX15.2 (ROW)
- new net: D44.2 (A), MX44.2 (ROW)
- new net: D10.2 (A), MX10.2 (ROW)
- new net: D3.2 (A), MX3.2 (ROW)
- new net: D50.2 (A), MX50.2 (ROW)
- new net: D37.2 (A), MX37.2 (ROW)
- new net: D1.2 (A), MX1.2 (ROW)
- new net: D42.2 (A), MX42.2 (ROW)
- new net: D23.2 (A), MX23.2 (ROW)
- new net: D19.2 (A), MX19.2 (ROW)
- new net COL0: MX1.1 (COL), MX2.1 (COL), MX3.1 (COL), MX4.1 (COL), MX5.1 (COL), MX6.1 (COL), MX7.1 (COL), MX8.1 (COL)
- new net COL1: MX10.1 (COL), MX11.1 (COL), MX12.1 (COL), MX13.1 (COL), MX14.1 (COL), MX15.1 (COL), MX16.1 (COL), MX9.1 (COL)
- new net COL2: MX17.1 (COL), MX18.1 (COL), MX19.1 (COL), MX20.1 (COL), MX21.1 (COL), MX22.1 (COL), MX23.1 (COL), MX24.1 (COL)
- new net COL3: MX25.1 (COL), MX50.1 (COL)
- new net COL4: MX26.1 (COL), MX27.1 (COL), MX28.1 (COL), MX29.1 (COL), MX30.1 (COL), MX31.1 (COL), MX32.1 (COL), MX33.1 (COL)
- new net COL5: MX34.1 (COL), MX35.1 (COL), MX36.1 (COL), MX37.1 (COL), MX38.1 (COL), MX39.1 (COL), MX40.1 (COL), MX41.1 (COL)
- new net COL6: MX42.1 (COL), MX43.1 (COL), MX44.1 (COL), MX45.1 (COL), MX46.1 (COL), MX47.1 (COL), MX48.1 (COL), MX49.1 (COL)
- new net ROW0: D1.1 (K), D17.1 (K), D26.1 (K), D34.1 (K), D42.1 (K), D9.1 (K)
- new net ROW1: D10.1 (K), D18.1 (K), D2.1 (K), D27.1 (K), D35.1 (K), D43.1 (K)
- new net ROW2: D11.1 (K), D19.1 (K), D28.1 (K), D3.1 (K), D36.1 (K), D44.1 (K)
- new net ROW3: D12.1 (K), D20.1 (K), D25.1 (K), D29.1 (K), D37.1 (K), D4.1 (K), D45.1 (K)
- new net ROW4: D16.1 (K), D24.1 (K), D33.1 (K), D41.1 (K), D49.1 (K), D50.1 (K), D8.1 (K)
- new net ROW5: D15.1 (K), D23.1 (K), D32.1 (K), D40.1 (K), D48.1 (K), D7.1 (K)
- new net ROW6: D14.1 (K), D22.1 (K), D31.1 (K), D39.1 (K), D47.1 (K), D6.1 (K)
- new net ROW7: D13.1 (K), D21.1 (K), D30.1 (K), D38.1 (K), D46.1 (K), D5.1 (K)
Other:
- note added: "20 August 2023"
- note added: "Tenet Keyboard"
- moved on the sheet: C1, C2, C3, C4, C5, C6, C7, R1, R2, R3, R4, SW1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

Commit message: footprints assigned
Parts:
- C1, C2, C3, C4, C5, C6, C7: footprint (none) -> Capacitor_SMD:C_0805_2012Metric
- D1, D10, D11, D12, D13, D14, D15, D16, D17, D18, D19, D2, D20, D21, D22, D23, D24, D25, D26, D27, D28, D29, D3, D30, D31, D32, D33, D34, D35, D36, D37, D38, D39, D4, D40, D41, D42, D43, D44, D45, D46, D47, D48, D49, D5, D50, D6, D7, D8, D9: footprint (none) -> Diode_SMD:D_SOD-123
- MX1, MX10, MX11, MX12, MX13, MX14, MX15, MX16, MX17, MX18, MX19, MX2, MX20, MX21, MX22, MX23, MX24, MX26, MX27, MX28, MX29, MX3, MX30, MX31, MX32, MX33, MX34, MX35, MX36, MX37, MX38, MX39, MX4, MX40, MX41, MX42, MX43, MX44, MX45, MX46, MX47, MX48, MX49, MX5, MX6, MX7, MX8, MX9: footprint (none) -> Kailh_Choc:KailhChoc-1U
- MX25, MX50: footprint (none) -> Kailh_Choc:KailhChoc-1.75U
- R1, R2, R3, R4: footprint (none) -> Resistor_SMD:R_0805_2012Metric
- SW1: footprint (none) -> random-keyboard-parts.pretty-master:SKQG-1155865
- Y1: footprint (none) -> Crystal:Crystal_SMD_3225-4Pin_3.2x2.5mm

Commit message: pcb 1, mostly done
Parts:
- removed C1: 1µF, Capacitor_SMD:C_0805_2012Metric, symbol Device:C_Small
- removed C2, C3, C4: 0.1µF, Capacitor_SMD:C_0805_2012Metric, symbol Device:C_Small
- removed C5: 10µF, Capacitor_SMD:C_0805_2012Metric, symbol Device:C_Small
- removed C6, C7: 22pF, Capacitor_SMD:C_0805_2012Metric, symbol Device:C_Small
- removed R1, R4: 10kΩ, Resistor_SMD:R_0805_2012Metric, symbol Device:R_Small
- removed R2, R3: 22Ω, Resistor_SMD:R_0805_2012Metric, symbol Device:R_Small
- removed SW1: SW_Push, random-keyboard-parts.pretty-master:SKQG-1155865, symbol Switch:SW_Push
- removed U1: ATmega32U4-A, Package_QFP:TQFP-44_10x10mm_P0.8mm, symbol MCU_Microchip_ATmega:ATmega32U4-A
- removed Y1: 16MHz, Crystal:Crystal_SMD_3225-4Pin_3.2x2.5mm, symbol Device:Crystal_GND24_Small
- added U1: kb2040, kb2040:kb2040, symbol kb2040:kb2040
- MX1, MX10, MX11, MX12, MX13, MX14, MX15, MX16, MX17, MX18, MX19, MX2, MX20, MX21, MX22, MX23, MX24, MX26, MX27, MX28, MX29, MX3, MX30, MX31, MX32, MX33, MX34, MX35, MX36, MX37, MX38, MX39, MX4, MX40, MX41, MX42, MX43, MX44, MX45, MX46, MX47, MX48, MX49, MX5, MX6, MX7, MX8, MX9: footprint Kailh_Choc:KailhChoc-1U -> keyswitches.pretty-master:Kailh_socket_PG1350
- MX25, MX50: footprint Kailh_Choc:KailhChoc-1.75U -> keyswitches.pretty-master:Kailh_socket_PG1350
Connections:
- net GND: now also U1.16 (GND), U1.4 (GND), U1.5 (GND)
